Commit message: New street file added, edited bot3 Model(Unstable)

File: catkin_ws/src/turtlebot3/turtlebot3_description/urdf/turtlebot3_burger.gazebo.xacro (robot description, xacro)
@@ -8,30 +8,30 @@
   </gazebo>
   <gazebo reference="wheel_left_link">
-    <mu1>0.1</mu1>
-    <mu2>0.1</mu2>
+    <mu1>0.2</mu1>
+    <mu2>0.2</mu2>
     <kp>500000.0</kp>
     <kd>10.0</kd>
     <minDepth>0.001</minDepth>
-    <maxVel>0.1</maxVel>
+    <maxVel>0.5</maxVel>
     <fdir1>1 0 0</fdir1>
     <material>Gazebo/FlatBlack</material>
   </gazebo>
   <gazebo reference="wheel_right_link">
-    <mu1>0.1</mu1>
-    <mu2>0.1</mu2>
+    <mu1>0.2</mu1>
+    <mu2>0.2</mu2>
     <kp>500000.0</kp>
     <kd>10.0</kd>
     <minDepth>0.001</minDepth>
-    <maxVel>0.1</maxVel>
+    <maxVel>0.5</maxVel>
     <fdir1>1 0 0</fdir1>
     <material>Gazebo/FlatBlack</material>
   </gazebo>
   <gazebo reference="caster_back_link">
-    <mu1>0.1</mu1>
-    <mu2>0.1</mu2>
+    <mu1>0.2</mu1>
+    <mu2>0.2</mu2>
     <kp>1000000.0</kp>
     <kd>100.0</kd>
     <minDepth>0.001</minDepth>
-    <maxVel>1.0</maxVel>
+    <maxVel>5.0</maxVel>
     <material>Gazebo/FlatBlack</material>
   </gazebo>

File: catkin_ws/src/turtlebot3/turtlebot3_description/urdf/turtlebot3_burger.urdf.xacro (robot description, xacro)
@@ -7,26 +7,26 @@
     <parent link="base_footprint"/>
     <child link="base_link"/>
-    <origin xyz="0.0 0.0 0.010" rpy="0 0 0"/>
+    <origin xyz="0.0 0.0 0.050" rpy="0 0 0"/>
   </joint>
   <link name="base_link">
     <visual>
-      <origin xyz="-0.032 0 0.0" rpy="0 0 0"/>
+      <origin xyz="-0.16 0 0.0" rpy="0 0 0"/>
       <geometry>
-        <mesh filename="package://turtlebot3_description/meshes/bases/burger_base.stl" scale="0.001 0.001 0.001"/>
+        <mesh filename="package://turtlebot3_description/meshes/bases/burger_base.stl" scale="0.005 0.005 0.005"/>
       </geometry>
       <material name="light_black"/>
     </visual>
     <collision>
-      <origin xyz="-0.032 0 0.070" rpy="0 0 0"/>
+      <origin xyz="-0.16 0 0.35" rpy="0 0 0"/>
       <geometry>
-        <box size="0.140 0.140 0.143"/>
+        <box size="0.7 0.7 0.715"/>
       </geometry>
     </collision>
     <inertial>
       <origin xyz="0 0 0" rpy="0 0 0"/>
-      <mass value="8.2573504e-01"/>
-      <inertia ixx="2.2124416e-03" ixy="-1.2294101e-05" ixz="3.4938785e-05"
-               iyy="2.1193702e-03" iyz="-5.0120904e-06"
-               izz="2.0064271e-03" />
+      <mass value="103.2125"/>
+      <inertia ixx="0.2765" ixy="-1.53675e-03" ixz="4.36725e-03"
+               iyy="0.2649125" iyz="-6.2651125e-04"
+               izz="0.2508" />
     </inertial>
   </link>
@@ -34,5 +34,5 @@
     <parent link="base_link"/>
     <child link="wheel_left_link"/>
-    <origin xyz="0.0 0.08 0.023" rpy="-1.57 0 0"/>
+    <origin xyz="0.0 0.4 0.115" rpy="-1.57 0 0"/>
     <axis xyz="0 0 1"/>
   </joint>
@@ -41,5 +41,5 @@
       <origin xyz="0 0 0" rpy="1.57 0 0"/>
       <geometry>
-        <mesh filename="package://turtlebot3_description/meshes/wheels/left_tire.stl" scale="0.001 0.001 0.001"/>
+        <mesh filename="package://turtlebot3_description/meshes/wheels/left_tire.stl" scale="0.005 0.005 0.005"/>
       </geometry>
       <material name="dark"/>
@@ -48,13 +48,13 @@
       <origin xyz="0 0 0" rpy="0 0 0"/>
       <geometry>
-        <cylinder length="0.018" radius="0.033"/>
+        <cylinder length="0.09" radius="0.165"/>
       </geometry>
     </collision>
     <inertial>
       <origin xyz="0 0 0" />
-      <mass value="2.8498940e-02" />
-      <inertia ixx="1.1175580e-05" ixy="-4.2369783e-11" ixz="-5.9381719e-09"
-               iyy="1.1192413e-05" iyz="-1.4400107e-11"
-               izz="2.0712558e-05" />
+      <mass value="3.5623675" />
+      <inertia ixx="1.3969475e-03" ixy="-5.296222875e-09" ixz="-7.4225e-07"
+               iyy="1.399051625e-03" iyz="-1.800013375e-09"
+               izz="2.58906975e-03" />
       </inertial>
   </link>
@@ -62,5 +62,5 @@
     <parent link="base_link"/>
     <child link="wheel_right_link"/>
-    <origin xyz="0.0 -0.080 0.023" rpy="-1.57 0 0"/>
+    <origin xyz="0.0 -0.4 0.115" rpy="-1.57 0 0"/>
     <axis xyz="0 0 1"/>
   </joint>
@@ -69,5 +69,5 @@
       <origin xyz="0 0 0" rpy="1.57 0 0"/>
       <geometry>
-        <mesh filename="package://turtlebot3_description/meshes/wheels/right_tire.stl" scale="0.001 0.001 0.001"/>
+        <mesh filename="package://turtlebot3_description/meshes/wheels/right_tire.stl" scale="0.005 0.005 0.005"/>
       </geometry>
       <material name="dark"/>
@@ -76,13 +76,13 @@
       <origin xyz="0 0 0" rpy="0 0 0"/>
       <geometry>
-        <cylinder length="0.018" radius="0.033"/>
+        <cylinder length="0.09" radius="0.165"/>
       </geometry>
     </collision>
     <inertial>
       <origin xyz="0 0 0" />
-      <mass value="2.8498940e-02" />
-      <inertia ixx="1.1175580e-05" ixy="-4.2369783e-11" ixz="-5.9381719e-09"
-               iyy="1.1192413e-05" iyz="-1.4400107e-11"
-               izz="2.0712558e-05" />
+      <mass value="3.5623675" />
+      <inertia ixx="1.3969475e-03" ixy="-5.296222875e-09" ixz="-7.4225e-07"
+               iyy="1.399051625e-03" iyz="-1.800013375e-09"
+               izz="2.58906975e-03" />
       </inertial>
   </link>
@@ -90,5 +90,5 @@
     <parent link="base_link"/>
     <child link="caster_back_link"/>
-    <origin xyz="-0.081 0 -0.004" rpy="-1.57 0 0"/>
+    <origin xyz="-0.405 0 -0.02" rpy="-1.57 0 0"/>
   </joint>
   <link name="caster_back_link">
@@ -96,13 +96,13 @@
       <origin xyz="0 0.001 0" rpy="0 0 0"/>
       <geometry>
-        <box size="0.030 0.009 0.020"/>
+        <box size="0.15 0.045 0.100"/>
       </geometry>
     </collision>
     <inertial>
       <origin xyz="0 0 0" />
-      <mass value="0.005" />
-      <inertia ixx="0.001" ixy="0.0" ixz="0.0"
-               iyy="0.001" iyz="0.0"
-               izz="0.001" />
+      <mass value="6.25" />
+      <inertia ixx="0.125" ixy="0.0" ixz="0.0"
+               iyy="0.125" iyz="0.0"
+               izz="0.125" />
     </inertial>
   </link>
@@ -110,5 +110,5 @@
     <parent link="base_link"/>
     <child link="imu_link"/>
-    <origin xyz="-0.032 0 0.068" rpy="0 0 0"/>
+    <origin xyz="-0.16 0 0.34" rpy="0 0 0"/>
   </joint>
   <link name="imu_link"/>
@@ -116,5 +116,5 @@
     <parent link="base_link"/>
     <child link="base_scan"/>
-    <origin xyz="-0.032 0 0.172" rpy="0 0 0"/>
+    <origin xyz="-0.16 0 0.86" rpy="0 0 0"/>
   </joint>
   <link name="base_scan">
@@ -122,20 +122,20 @@
       <origin xyz="0 0 0.0" rpy="0 0 0"/>
       <geometry>
-        <mesh filename="package://turtlebot3_description/meshes/sensors/lds.stl" scale="0.001 0.001 0.001"/>
+        <mesh filename="package://turtlebot3_description/meshes/sensors/lds.stl" scale="0.005 0.005 0.005"/>
       </geometry>
       <material name="dark"/>
     </visual>
     <collision>
-      <origin xyz="0.015 0 -0.0065" rpy="0 0 0"/>
+      <origin xyz="0.075 0 -0.0325" rpy="0 0 0"/>
       <geometry>
-        <cylinder length="0.0315" radius="0.055"/>
+        <cylinder length="0.1575" radius="0.275"/>
       </geometry>
     </collision>
     <inertial>
-      <mass value="0.114" />
+      <mass value="0.57" />
       <origin xyz="0 0 0" />
-      <inertia ixx="0.001" ixy="0.0" ixz="0.0"
-               iyy="0.001" iyz="0.0"
-               izz="0.001" />
+      <inertia ixx="0.005" ixy="0.0" ixz="0.0"
+               iyy="0.005" iyz="0.0"
+               izz="0.005" />
     </inertial>
   </link>
@@ -143,24 +143,24 @@
     <parent link="base_link"/>
     <child link="camera_link"/>
-    <origin xyz="0.02 0 0.171" rpy="0 0 0"/>
+    <origin xyz="0.1 0 0.855" rpy="0 0 0"/>
   </joint>
 <link name='camera_link'>
 <inertial>
   <origin xyz="0 0 0.0" rpy="0 0 0"/>
-  <inertia ixx="0.001" ixy="0.0" ixz="0.0"
-           iyy="0.001" iyz="0.0"
-           izz="0.001" />
-  <mass value="0.004" />
+  <inertia ixx="0.005" ixy="0.0" ixz="0.0"
+           iyy="0.005" iyz="0.0"
+           izz="0.005" />
+  <mass value="0.02" />
 </inertial>
 <visual name='camera_visual'>
-    <origin xyz="0.02 -0.01 -0.02" rpy="0 1.57 0"/>
+    <origin xyz="0.1 -0.05 -0.1" rpy="0 1.57 0"/>
   <geometry>
-    <mesh filename="package://turtlebot3_description/meshes/sensors/ras_cam.dae" scale="1 1 1"/>
+    <mesh filename="package://turtlebot3_description/meshes/sensors/ras_cam.dae" scale="5 5 5"/>
   </geometry>
 </visual>
 <collision name='camera_collision'>
-  <pose frame=''>0.02 -0.01 0.105 0 -0 0</pose>
+  <pose frame=''>0.1 -0.05 0.525 0 -0 0</pose>
   <geometry>
-     <box size="0.003 0.03 0.025"/>
+     <box size="0.015 0.015 0.125"/>
   </geometry>
 </collision>

Commit message: Updated Models, generating stuff

File: catkin_ws/src/turtlebot3/turtlebot3_description/urdf/turtlebot3_burger.gazebo.xacro (robot description, xacro)
@@ -8,6 +8,6 @@
   </gazebo>
   <gazebo reference="wheel_left_link">
-    <mu1>0.2</mu1>
-    <mu2>0.2</mu2>
+    <mu1>0.1</mu1>
+    <mu2>0.1</mu2>
     <kp>500000.0</kp>
     <kd>10.0</kd>
@@ -18,6 +18,6 @@
   </gazebo>
   <gazebo reference="wheel_right_link">
-    <mu1>0.2</mu1>
-    <mu2>0.2</mu2>
+    <mu1>0.1</mu1>
+    <mu2>0.1</mu2>
     <kp>500000.0</kp>
     <kd>10.0</kd>
@@ -28,6 +28,6 @@
   </gazebo>
   <gazebo reference="caster_back_link">
-    <mu1>0.2</mu1>
-    <mu2>0.2</mu2>
+    <mu1>0.1</mu1>
+    <mu2>0.1</mu2>
     <kp>1000000.0</kp>
     <kd>100.0</kd>
@@ -58,5 +58,5 @@
       <leftJoint>wheel_left_joint</leftJoint>
       <rightJoint>wheel_right_joint</rightJoint>
-      <wheelSeparation>0.160</wheelSeparation>
+      <wheelSeparation>0.16</wheelSeparation>
       <wheelDiameter>0.066</wheelDiameter>
       <wheelAcceleration>1</wheelAcceleration>
@@ -131,6 +131,6 @@
     <horizontal_fov>1.3962634</horizontal_fov>
     <image>
-      <width>2000</width>
-      <height>800</height>
+      <width>1280</width>
+      <height>384</height>
       <format>R8G8B8</format>
     </image>

File: catkin_ws/src/turtlebot3/turtlebot3_description/urdf/turtlebot3_burger.urdf.xacro (robot description, xacro)
@@ -96,9 +96,15 @@
   <link name="caster_back_link">
     <collision>
-      <origin xyz="0 0.001 0" rpy="0 0 0"/>
+      <origin xyz="0 0.005 0" rpy="0 0 0"/>
       <geometry>
         <box size="0.15 0.045 0.100"/>
       </geometry>
     </collision>
+    <visual>
+      <origin xyz="0 0.005 0" rpy="0 0 0"/>
+      <geometry>
+        <box size="0.15 0.045 0.100"/>
+      </geometry>
+    </visual>
     <inertial>
       <origin xyz="0 0 0" />
@@ -148,5 +154,5 @@
   </joint>
 <link name='camera_link'>
-<inertial>
+<!-- <inertial>
   <origin xyz="0 0 0.0" rpy="0 0 0"/>
   <inertia ixx="0.005" ixy="0.0" ixz="0.0"
@@ -154,5 +160,5 @@
            izz="0.005" />
   <mass value="0.02" />
-</inertial>
+</inertial> -->
 <visual name='camera_visual'>
     <origin xyz="0.1 -0.05 -0.1" rpy="0 1.57 0"/>

Commit message: Updated Camera Numbers to Three

File: catkin_ws/src/turtlebot3/turtlebot3_description/urdf/turtlebot3_burger.gazebo.xacro (robot description, xacro)
@@ -164,3 +164,81 @@
 </sensor>
 </gazebo>
+  <gazebo reference="camera_link_2">
+<sensor type="camera" name="camera2">
+  <update_rate>15.0</update_rate>
+  <camera name="head">
+    <horizontal_fov>1.3962634</horizontal_fov>
+    <image>
+      <width>1280</width>
+      <height>384</height>
+      <format>R8G8B8</format>
+    </image>
+    <clip>
+      <near>0.02</near>
+      <far>300</far>
+    </clip>
+    <noise>
+      <type>gaussian</type>
+      <!-- Noise is sampled independently per pixel on each frame.
+           That pixel's noise value is added to each of its color
+           channels, which at that point lie in the range [0,1]. -->
+      <mean>0.0</mean>
+      <stddev>0.007</stddev>
+    </noise>
+  </camera>
+  <plugin name="camera_controller" filename="libgazebo_ros_camera.so">
+    <alwaysOn>true</alwaysOn>
+    <updateRate>0.0</updateRate>
+    <cameraName>rrbot/camera2</cameraName>
+    <imageTopicName>image_raw</imageTopicName>
+    <cameraInfoTopicName>camera_info</cameraInfoTopicName>
+    <frameName>camera_link</frameName>
+    <hackBaseline>0.07</hackBaseline>
+    <distortionK1>0.0</distortionK1>
+    <distortionK2>0.0</distortionK2>
+    <distortionK3>0.0</distortionK3>
+    <distortionT1>0.0</distortionT1>
+    <distortionT2>0.0</distortionT2>
+  </plugin>
+</sensor>
+</gazebo>
+  <gazebo reference="camera_link_3">
+<sensor type="camera" name="camera3">
+  <update_rate>15.0</update_rate>
+  <camera name="head">
+    <horizontal_fov>1.3962634</horizontal_fov>
+    <image>
+      <width>1280</width>
+      <height>384</height>
+      <format>R8G8B8</format>
+    </image>
+    <clip>
+      <near>0.02</near>
+      <far>300</far>
+    </clip>
+    <noise>
+      <type>gaussian</type>
+      <!-- Noise is sampled independently per pixel on each frame.
+           That pixel's noise value is added to each of its color
+           channels, which at that point lie in the range [0,1]. -->
+      <mean>0.0</mean>
+      <stddev>0.007</stddev>
+    </noise>
+  </camera>
+  <plugin name="camera_controller" filename="libgazebo_ros_camera.so">
+    <alwaysOn>true</alwaysOn>
+    <updateRate>0.0</updateRate>
+    <cameraName>rrbot/camera3</cameraName>
+    <imageTopicName>image_raw</imageTopicName>
+    <cameraInfoTopicName>camera_info</cameraInfoTopicName>
+    <frameName>camera_link</frameName>
+    <hackBaseline>0.07</hackBaseline>
+    <distortionK1>0.0</distortionK1>
+    <distortionK2>0.0</distortionK2>
+    <distortionK3>0.0</distortionK3>
+    <distortionT1>0.0</distortionT1>
+    <distortionT2>0.0</distortionT2>
+  </plugin>
+</sensor>
+</gazebo>
 </robot>

File: catkin_ws/src/turtlebot3/turtlebot3_description/urdf/turtlebot3_burger.urdf.xacro (robot description, xacro)
@@ -174,3 +174,55 @@
 </collision>
 </link>
+  <joint name="camera_joint_2" type="fixed">
+    <parent link="base_link"/>
+    <child link="camera_link_2"/>
+    <origin xyz="0.056 0 0.4788" rpy="0 0 0.785"/>
+  </joint>
+<link name='camera_link_2'>
+<!-- <inertial>
+  <origin xyz="0 0 0.0" rpy="0 0 0"/>
+  <inertia ixx="0.005" ixy="0.0" ixz="0.0"
+           iyy="0.005" iyz="0.0"
+           izz="0.005" />
+  <mass value="0.02" />
+</inertial> -->
+<visual name='camera_visual_2'>
+    <origin xyz="0.056 -0.028 -0.056" rpy="0 1.57 0"/>
+  <geometry>
+    <mesh filename="package://turtlebot3_description/meshes/sensors/ras_cam.dae" scale="2.8 2.8 2.8"/>
+  </geometry>
+</visual>
+<collision name='camera_collision_2'>
+  <pose frame=''>0.056 -0.028 -0.056 0 -0 0</pose>
+  <geometry>
+     <box size="0.0084 0.084 0.07"/>
+  </geometry>
+</collision>
+</link>
+  <joint name="camera_joint_3" type="fixed">
+    <parent link="base_link"/>
+    <child link="camera_link_3"/>
+    <origin xyz="0.056 0 0.4788" rpy="0 0 -0.785"/>
+  </joint>
+<link name='camera_link_3'>
+<!-- <inertial>
+  <origin xyz="0 0 0.0" rpy="0 0 0"/>
+  <inertia ixx="0.005" ixy="0.0" ixz="0.0"
+           iyy="0.005" iyz="0.0"
+           izz="0.005" />
+  <mass value="0.02" />
+</inertial> -->
+<visual name='camera_visual_3'>
+    <origin xyz="0.056 -0.028 -0.056" rpy="0 1.57 0"/>
+  <geometry>
+    <mesh filename="package://turtlebot3_description/meshes/sensors/ras_cam.dae" scale="2.8 2.8 2.8"/>
+  </geometry>
+</visual>
+<collision name='camera_collision_3'>
+  <pose frame=''>0.056 -0.028 -0.056 0 -0 0</pose>
+  <geometry>
+     <box size="0.0084 0.084 0.07"/>
+  </geometry>
+</collision>
+</link>
 </robot>
